File: pcb/modular_device_teensy.sch (KiCad schematic (older format))
At the start: 11 parts, among them P1 PWR_JACK_2.5x5.5_SMD_RA, P2 HEADER_01X03_SMD_RA, P3 HEADER_01X03_SMD_RA, P4 HEADER_01X03_SMD_RA, P5 BNC_DOUBLE_RA

Commit message: Added some components.
Parts:
- removed D1, D2: diode_schottky_40V_1A, footprints:DO-214AC(SMA), symbol diode_schottky_40V_1A
- added D1, D2: diode_schottky_15V_1A, modular_device_teensy:DO-214BA, symbol diode_schottky_15V_1A
- C1, C2: footprint footprints:SM1210 -> modular_device_teensy:SM1210
- P1: footprint footprints:DCJACK_2PIN_HIGHCURRENT_SMD_RA -> modular_device_teensy:DCJACK_2PIN_HIGHCURRENT_SMD_RA
- P2, P3, P4: footprint footprints:Header_3_Pin_SMD_RA -> modular_device_teensy:Header_3_Pin_SMD_RA
- P5: footprint footprints:BNC_DOUBLE -> modular_device_teensy:BNC_DOUBLE
- REG1: footprint footprints:DC_DC_CONV_R78C -> modular_device_teensy:DC_DC_CONV_R78C
- TEENSY1: footprint footprints:TEENSY_3 -> modular_device_teensy:TEENSY_3
Changed lines of the file:
@@
 F 0 "TEENSY1" H 3250 3747 60  0000 C CNN
 F 1 "TEENSY_3_2" H 3250 3641 60  0000 C CNN
-F 2 "footprints:TEENSY_3" H 3250 3800 60  0001 C CNN
+F 2 "modular_device_teensy:TEENSY_3" H 3250 3800 60  0001 C CNN
 F 3 "" H 3300 5500 60  0000 C CNN
 F 4 "digikey" H 3250 3900 60  0001 C CNN "Vendor"
@@
 F 0 "REG1" H 3250 7397 60  0000 C CNN
 F 1 "CONV_DC_DC_5V_1A" H 3250 7291 60  0000 C CNN
-F 2 "footprints:DC_DC_CONV_R78C" H 3350 6750 60  0001 C CNN
+F 2 "modular_device_teensy:DC_DC_CONV_R78C" H 3350 6750 60  0001 C CNN
 F 3 "" H 3250 7150 60  0000 C CNN
 F 4 "digikey" H 3250 6950 60  0001 C CNN "Vendor"
@@
 F 0 "C1" H 2765 7480 40  0000 L CNN
 F 1 "10uF" H 2650 7450 30  0000 C CNN
-F 2 "footprints:SM1210" H 2688 7300 30  0001 C CNN
+F 2 "modular_device_teensy:SM1210" H 2688 7300 30  0001 C CNN
 F 3 "" H 2650 7450 60  0000 C CNN
 F 4 "digikey" H 2750 7650 60  0001 C CNN "Vendor"
@@
 F 0 "C2" H 3965 7480 40  0000 L CNN
 F 1 "10uF" H 3850 7450 30  0000 C CNN
-F 2 "footprints:SM1210" H 3888 7300 30  0001 C CNN
+F 2 "modular_device_teensy:SM1210" H 3888 7300 30  0001 C CNN
 F 3 "" H 3850 7450 60  0000 C CNN
 F 4 "digikey" H 3950 7650 60  0001 C CNN "Vendor"
@@
 	3850 7100 3850 7250
 $Comp
-L GND #PWR9
+L GND #PWR01
 U 1 1 5751CFDE
 P 3250 7750
-F 0 "#PWR9" H 3250 7500 50  0001 C CNN
+F 0 "#PWR01" H 3250 7500 50  0001 C CNN
 F 1 "GND" H 3255 7577 50  0000 C CNN
 F 2 "" H 3250 7750 50  0000 C CNN
@@
 F 0 "P1" H 1450 7600 50  0000 C CNN
 F 1 "PWR_JACK_2.5x5.5_SMD_RA" V 1550 7450 50  0000 C CNN
-F 2 "footprints:DCJACK_2PIN_HIGHCURRENT_SMD_RA" H 1350 7500 60  0001 C CNN
+F 2 "modular_device_teensy:DCJACK_2PIN_HIGHCURRENT_SMD_RA" H 1350 7500 60  0001 C CNN
 F 3 "" H 1450 7600 60  0000 C CNN
 F 4 "digikey" H 1550 7700 60  0001 C CNN "Vendor"
@@
 $EndComp
 $Comp
-L PWR_FLAG #FLG2
+L PWR_FLAG #FLG02
 U 1 1 5751E700
 P 700 7400
-F 0 "#FLG2" H 700 7495 50  0001 C CNN
+F 0 "#FLG02" H 700 7495 50  0001 C CNN
 F 1 "PWR_FLAG" H 700 7624 50  0000 C CNN
 F 2 "" H 700 7400 50  0000 C CNN
@@
 $EndComp
 $Comp
-L PWR_FLAG #FLG1
+L PWR_FLAG #FLG03
 U 1 1 5751E72B
 P 1000 7300
-F 0 "#FLG1" H 1000 7395 50  0001 C CNN
+F 0 "#FLG03" H 1000 7395 50  0001 C CNN
 F 1 "PWR_FLAG" H 1000 7524 50  0000 C CNN
 F 2 "" H 1000 7300 50  0000 C CNN
@@
 $EndComp
 $Comp
-L VAA #PWR6
+L VAA #PWR04
 U 1 1 5751E779
 P 1150 7350
-F 0 "#PWR6" H 1150 7200 50  0001 C CNN
+F 0 "#PWR04" H 1150 7200 50  0001 C CNN
 F 1 "VAA" H 1167 7523 50  0000 C CNN
 F 2 "" H 1150 7350 50  0000 C CNN
@@
 	700  7500 1250 7500
 $Comp
-L GND #PWR7
+L GND #PWR05
 U 1 1 5751E825
 P 1150 7550
-F 0 "#PWR7" H 1150 7300 50  0001 C CNN
+F 0 "#PWR05" H 1150 7300 50  0001 C CNN
 F 1 "GND" H 1155 7377 50  0000 C CNN
 F 2 "" H 1150 7550 50  0000 C CNN
@@
 Connection ~ 1150 7500
 $Comp
-L GND #PWR3
+L GND #PWR06
 U 1 1 5751EC8F
 P 1500 2200
-F 0 "#PWR3" H 1500 1950 50  0001 C CNN
+F 0 "#PWR06" H 1500 1950 50  0001 C CNN
 F 1 "GND" H 1505 2027 50  0000 C CNN
 F 2 "" H 1500 2200 50  0000 C CNN
@@
 F 0 "P2" H 1100 5900 50  0000 C CNN
 F 1 "HEADER_01X03_SMD_RA" V 1200 6100 50  0000 C CNN
-F 2 "footprints:Header_3_Pin_SMD_RA" H 1000 6200 60  0001 C CNN
+F 2 "modular_device_teensy:Header_3_Pin_SMD_RA" H 1000 6200 60  0001 C CNN
 F 3 "" H 1100 6300 60  0000 C CNN
 F 4 "digikey" H 1200 6400 60  0001 C CNN "Vendor"
@@
 F 0 "P3" H 1700 5900 50  0000 C CNN
 F 1 "HEADER_01X03_SMD_RA" V 1800 6100 50  0000 C CNN
-F 2 "footprints:Header_3_Pin_SMD_RA" H 1600 6200 60  0001 C CNN
+F 2 "modular_device_teensy:Header_3_Pin_SMD_RA" H 1600 6200 60  0001 C CNN
 F 3 "" H 1700 6300 60  0000 C CNN
 F 4 "digikey" H 1800 6400 60  0001 C CNN "Vendor"
@@
 F 0 "P4" H 2300 5900 50  0000 C CNN
 F 1 "HEADER_01X03_SMD_RA" V 2400 6100 50  0000 C CNN
-F 2 "footprints:Header_3_Pin_SMD_RA" H 2200 6200 60  0001 C CNN
+F 2 "modular_device_teensy:Header_3_Pin_SMD_RA" H 2200 6200 60  0001 C CNN
 F 3 "" H 2300 6300 60  0000 C CNN
 F 4 "digikey" H 2400 6400 60  0001 C CNN "Vendor"
@@
 GND
 $Comp
-L VAA #PWR4
+L VAA #PWR07
 U 1 1 5751F3BD
 P 2650 7100
-F 0 "#PWR4" H 2650 6950 50  0001 C CNN
+F 0 "#PWR07" H 2650 6950 50  0001 C CNN
 F 1 "VAA" H 2667 7273 50  0000 C CNN
 F 2 "" H 2650 7100 50  0000 C CNN
@@
 F 0 "P5" H 5500 7665 50  0000 C CNN
 F 1 "BNC_DOUBLE_RA" H 5500 7574 50  0000 C CNN
-F 2 "footprints:BNC_DOUBLE" H 5500 6200 60  0001 C CNN
+F 2 "modular_device_teensy:BNC_DOUBLE" H 5500 6200 60  0001 C CNN
 F 3 "" H 5500 6200 60  0000 C CNN
 F 4 "digikey" H 5600 7650 60  0001 C CNN "Vendor"
@@
 $EndComp
 $Comp
-L GND #PWR8
+L GND #PWR08
 U 1 1 5751FC2B
 P 5850 7550
-F 0 "#PWR8" H 5850 7300 50  0001 C CNN
+F 0 "#PWR08" H 5850 7300 50  0001 C CNN
 F 1 "GND" H 5855 7377 50  0000 C CNN
 F 2 "" H 5850 7550 50  0000 C CNN
@@
 Text Label 4900 7450 0    60   ~ 0
 BNC_B
-$Comp
-L diode_schottky_40V_1A D1
-U 1 1 57520086
-P 4350 1950
-F 0 "D1" V 4350 1882 50  0000 R CNN
-F 1 "diode_schottky_40V_1A" H 4070 1870 50  0001 L CNN
-F 2 "footprints:DO-214AC(SMA)" H 4200 1930 60  0001 C CNN
-F 3 "" H 4300 2030 60  0001 C CNN
-F 4 "digikey" H 4400 2130 60  0001 C CNN "Vendor"
-F 5 "SS14CT-ND" H 4500 2230 60  0001 C CNN "PartNumber"
-F 6 "DIODE SCHOTTKY 40V 1A SMA" H 4600 2330 60  0001 C CNN "Description"
-	1    4350 1950
-	0    -1   -1   0
-$EndComp
 Text Label 4350 1800 0    60   ~ 0
 V_USB
@@
 	4200 2100 4900 2100
 $Comp
-L +5V #PWR5
+L +5V #PWR09
 U 1 1 57520478
 P 3850 7100
-F 0 "#PWR5" H 3850 6950 50  0001 C CNN
+F 0 "#PWR09" H 3850 6950 50  0001 C CNN
 F 1 "+5V" H 3865 7273 50  0000 C CNN
 F 2 "" H 3850 7100 50  0000 C CNN
@@
 $EndComp
 Connection ~ 3850 7150
-$Comp
-L diode_schottky_40V_1A D2
-U 1 1 575206A4
-P 4700 1950
-F 0 "D2" V 4700 1882 50  0000 R CNN
-F 1 "diode_schottky_40V_1A" H 4420 1870 50  0001 L CNN
-F 2 "footprints:DO-214AC(SMA)" H 4550 1930 60  0001 C CNN
-F 3 "" H 4650 2030 60  0001 C CNN
-F 4 "digikey" H 4750 2130 60  0001 C CNN "Vendor"
-F 5 "SS14CT-ND" H 4850 2230 60  0001 C CNN "PartNumber"
-F 6 "DIODE SCHOTTKY 40V 1A SMA" H 4950 2330 60  0001 C CNN "Description"
-	1    4700 1950
-	0    -1   -1   0
-$EndComp
 Wire Wire Line
 	4700 2100 4700 2050
 Connection ~ 4350 2100
 $Comp
-L +5V #PWR1
+L +5V #PWR010
 U 1 1 57520888
 P 4700 1800
-F 0 "#PWR1" H 4700 1650 50  0001 C CNN
+F 0 "#PWR010" H 4700 1650 50  0001 C CNN
 F 1 "+5V" H 4715 1973 50  0000 C CNN
 F 2 "" H 4700 1800 50  0000 C CNN
@@
 NoConn ~ 4200 2300
 $Comp
-L VCC #PWR2
+L VCC #PWR011
 U 1 1 57520D74
 P 4900 1800
-F 0 "#PWR2" H 4900 1650 50  0001 C CNN
+F 0 "#PWR011" H 4900 1650 50  0001 C CNN
 F 1 "VCC" H 4917 1973 50  0000 C CNN
 F 2 "" H 4900 1800 50  0000 C CNN
@@
 	4900 2100 4900 1800
 Connection ~ 4700 2100
+$Comp
+L diode_schottky_15V_1A D1
+U 1 1 5764103B
+P 4350 1950
+F 0 "D1" V 4350 1882 50  0000 R CNN
+F 1 "diode_schottky_15V_1A" H 4070 1870 50  0001 L CNN
+F 2 "modular_device_teensy:DO-214BA" H 4200 1930 60  0001 C CNN
+F 3 "" H 4300 2030 60  0001 C CNN
+F 4 "digikey" H 4400 2130 60  0001 C CNN "Vendor"
+F 5 "LSM115JE3/TR13CT-ND" H 4500 2230 60  0001 C CNN "PartNumber"
+F 6 "DIODE SCHOTTKY 15V 1A DO214BA" H 4600 2330 60  0001 C CNN "Description"
+	1    4350 1950
+	0    -1   -1   0
+$EndComp
+$Comp
+L diode_schottky_15V_1A D2
+U 1 1 57640DFA
+P 4700 1950
+F 0 "D2" V 4700 1882 50  0000 R CNN
+F 1 "diode_schottky_15V_1A" H 4420 1870 50  0001 L CNN
+F 2 "modular_device_teensy:DO-214BA" H 4550 1930 60  0001 C CNN
+F 3 "" H 4650 2030 60  0001 C CNN
+F 4 "digikey" H 4750 2130 60  0001 C CNN "Vendor"
+F 5 "LSM115JE3/TR13CT-ND" H 4850 2230 60  0001 C CNN "PartNumber"
+F 6 "DIODE SCHOTTKY 15V 1A DO214BA" H 4950 2330 60  0001 C CNN "Description"
+	1    4700 1950
+	0    -1   -1   0
+$EndComp
 $EndSCHEMATC

Commit message: Progress towards board layout.
Parts:
- added P?: HEADER_01X02_SMD_RA, modular_device_teensy:Header_2_Pin_SMD_RA, symbol HEADER_01X02_SMD_RA
Connections:
- net labels added: VDD
- wire segments 46 -> 50
Changed lines of the file:
@@
 LIBS:components
 LIBS:modular_device_teensy
+LIBS:modular_device_teensy-cache
 EELAYER 25 0
 EELAYER END
@@
 	4250 2000 4200 2000
 NoConn ~ 4200 2300
-$Comp
-L VCC #PWR011
-U 1 1 57520D74
-P 4900 1800
-F 0 "#PWR011" H 4900 1650 50  0001 C CNN
-F 1 "VCC" H 4917 1973 50  0000 C CNN
-F 2 "" H 4900 1800 50  0000 C CNN
-F 3 "" H 4900 1800 50  0000 C CNN
-	1    4900 1800
-	1    0    0    -1
-$EndComp
 Wire Wire Line
 	4900 2100 4900 1800
@@
 	0    -1   -1   0
 $EndComp
+$Comp
+L HEADER_01X02_SMD_RA P?
+U 1 1 57643F2D
+P 2900 6100
+F 0 "P?" H 2900 5950 50  0000 C CNN
+F 1 "HEADER_01X02_SMD_RA" V 3000 6100 50  0000 C CNN
+F 2 "modular_device_teensy:Header_2_Pin_SMD_RA" H 2800 6150 50  0001 C CNN
+F 3 "" H 2900 6250 50  0000 C CNN
+F 4 "digikey" H 3000 6350 60  0001 C CNN "Vendor"
+F 5 "A100903CT-ND" H 3100 6450 60  0001 C CNN "PartNumber"
+F 6 "CONN HEADER 2POS R/A SMD GOLD" H 3200 6550 60  0001 C CNN "Description"
+	1    2900 6100
+	-1   0    0    1
+$EndComp
+$Comp
+L VDD #PWR?
+U 1 1 576452DC
+P 4900 1800
+F 0 "#PWR?" H 4900 1650 50  0001 C CNN
+F 1 "VDD" H 4917 1973 50  0000 C CNN
+F 2 "" H 4900 1800 50  0000 C CNN
+F 3 "" H 4900 1800 50  0000 C CNN
+	1    4900 1800
+	1    0    0    -1
+$EndComp
+$Comp
+L VCC #PWR?
+U 1 1 57645344
+P 3150 6000
+F 0 "#PWR?" H 3150 5850 50  0001 C CNN
+F 1 "VCC" H 3167 6173 50  0000 C CNN
+F 2 "" H 3150 6000 50  0000 C CNN
+F 3 "" H 3150 6000 50  0000 C CNN
+	1    3150 6000
+	1    0    0    -1
+$EndComp
+Wire Wire Line
+	3100 6050 3150 6050
+Wire Wire Line
+	3150 6050 3150 6000
+$Comp
+L GND #PWR?
+U 1 1 5764558A
+P 3150 6250
+F 0 "#PWR?" H 3150 6000 50  0001 C CNN
+F 1 "GND" H 3155 6077 50  0000 C CNN
+F 2 "" H 3150 6250 50  0000 C CNN
+F 3 "" H 3150 6250 50  0000 C CNN
+	1    3150 6250
+	1    0    0    -1
+$EndComp
+Wire Wire Line
+	3100 6150 3150 6150
+Wire Wire Line
+	3150 6150 3150 6250
 $EndSCHEMATC

Commit message: Added some components.
Parts:
- added D3, D4: diode_schottky_45V_10A, modular_device_teensy:CFP15, symbol diode_schottky_45V_10A
- added P7: HEADER_01X02_SMD_RA, modular_device_teensy:Header_2_Pin_SMD_RA, symbol HEADER_01X02_SMD_RA
- added SW1: KT_SWITCH, footprints:KT_SWITCH, symbol KT_SWITCH
- gave numbers to parts that had none: 1
Connections:
- net labels added: PROG, VEE
- wire segments 50 -> 67
- no-connect marks 1 -> 0
Other:
- moved on the sheet: P6

Commit message: More progress towards v1.0.
Parts:
- added MDT1: MODULAR_DEVICE_TEENSY_FEMALE, footprints:MODULAR_DEVICE_TEENSY_FEMALE, symbol MODULAR_DEVICE_TEENSY_FEMALE
Connections:
- net labels added: D10, D11, D12, D13, D14, D15, D16, D17, D18, D19, D2, D20, D21, D22, D23, D24, D25, D28, D29, D3, D30, D4, D5, D6, D9, DAC
- net labels removed: MISO, MOSI, SCK
- wire segments 67 -> 118
- no-connect marks 0 -> 5
Other:
- moved on the sheet: D1, D2, TEENSY1
