File: pcb/modular_device_teensy.sch (KiCad schematic (older format))
At the start: 17 parts, among them P1 PWR_JACK_2.5x5.5_SMD_RA, P2 HEADER_01X03_SMD_RA, P3 HEADER_01X03_SMD_RA, P4 HEADER_01X03_SMD_RA, P5 BNC_DOUBLE_RA, P6 HEADER_01X02_SMD_RA, P7 HEADER_01X02_SMD_RA, SW1 KT_SWITCH

Commit message: More progress towards v1.0.
Parts:
- added C3, C4, C5: 10uF, modular_device_teensy:SM1210, symbol 10uF
Connections:
- net 3V3: now also C5.1
- net GND: now also C3.2, C4.2, C5.2
- net VDD: now also C3.1
- net VEE: now also C4.1
Changed lines of the file:
@@
 	3850 7100 3850 7250
 $Comp
-L GND #PWR01
+L GND #PWR24
 U 1 1 5751CFDE
 P 3250 7750
-F 0 "#PWR01" H 3250 7500 50  0001 C CNN
+F 0 "#PWR24" H 3250 7500 50  0001 C CNN
 F 1 "GND" H 3255 7577 50  0000 C CNN
 F 2 "" H 3250 7750 50  0000 C CNN
@@
 $EndComp
 $Comp
-L PWR_FLAG #FLG02
+L PWR_FLAG #FLG6
 U 1 1 5751E700
 P 700 7400
-F 0 "#FLG02" H 700 7495 50  0001 C CNN
+F 0 "#FLG6" H 700 7495 50  0001 C CNN
 F 1 "PWR_FLAG" H 700 7624 50  0000 C CNN
 F 2 "" H 700 7400 50  0000 C CNN
@@
 $EndComp
 $Comp
-L PWR_FLAG #FLG03
+L PWR_FLAG #FLG5
 U 1 1 5751E72B
 P 1000 7300
-F 0 "#FLG03" H 1000 7395 50  0001 C CNN
+F 0 "#FLG5" H 1000 7395 50  0001 C CNN
 F 1 "PWR_FLAG" H 1000 7524 50  0000 C CNN
 F 2 "" H 1000 7300 50  0000 C CNN
@@
 $EndComp
 $Comp
-L VAA #PWR04
+L VAA #PWR21
 U 1 1 5751E779
 P 1150 7350
-F 0 "#PWR04" H 1150 7200 50  0001 C CNN
+F 0 "#PWR21" H 1150 7200 50  0001 C CNN
 F 1 "VAA" H 1167 7523 50  0000 C CNN
 F 2 "" H 1150 7350 50  0000 C CNN
@@
 	700  7500 1250 7500
 $Comp
-L GND #PWR05
+L GND #PWR22
 U 1 1 5751E825
 P 1150 7550
-F 0 "#PWR05" H 1150 7300 50  0001 C CNN
+F 0 "#PWR22" H 1150 7300 50  0001 C CNN
 F 1 "GND" H 1155 7377 50  0000 C CNN
 F 2 "" H 1150 7550 50  0000 C CNN
@@
 Connection ~ 1150 7500
 $Comp
-L GND #PWR06
+L GND #PWR3
 U 1 1 5751EC8F
 P 1500 2200
-F 0 "#PWR06" H 1500 1950 50  0001 C CNN
+F 0 "#PWR3" H 1500 1950 50  0001 C CNN
 F 1 "GND" H 1505 2027 50  0000 C CNN
 F 2 "" H 1500 2200 50  0000 C CNN
@@
 $EndComp
 $Comp
-L GND #PWR07
+L GND #PWR23
 U 1 1 5751FC2B
 P 5850 7550
-F 0 "#PWR07" H 5850 7300 50  0001 C CNN
+F 0 "#PWR23" H 5850 7300 50  0001 C CNN
 F 1 "GND" H 5855 7377 50  0000 C CNN
 F 2 "" H 5850 7550 50  0000 C CNN
@@
 	4800 2100 5750 2100
 $Comp
-L +5V #PWR08
+L +5V #PWR20
 U 1 1 57520478
 P 3850 7100
-F 0 "#PWR08" H 3850 6950 50  0001 C CNN
+F 0 "#PWR20" H 3850 6950 50  0001 C CNN
 F 1 "+5V" H 3865 7273 50  0000 C CNN
 F 2 "" H 3850 7100 50  0000 C CNN
@@
 Connection ~ 4950 2100
 $Comp
-L +5V #PWR09
+L +5V #PWR1
 U 1 1 57520888
 P 5300 1800
-F 0 "#PWR09" H 5300 1650 50  0001 C CNN
+F 0 "#PWR1" H 5300 1650 50  0001 C CNN
 F 1 "+5V" H 5315 1973 50  0000 C CNN
 F 2 "" H 5300 1800 50  0000 C CNN
@@
 $EndComp
 $Comp
-L VDD #PWR010
+L VDD #PWR14
 U 1 1 576452DC
 P 1850 5250
-F 0 "#PWR010" H 1850 5100 50  0001 C CNN
+F 0 "#PWR14" H 1850 5100 50  0001 C CNN
 F 1 "VDD" H 1867 5423 50  0000 C CNN
 F 2 "" H 1850 5250 50  0000 C CNN
@@
 $EndComp
 $Comp
-L VCC #PWR011
+L VCC #PWR15
 U 1 1 57645344
 P 2850 6000
-F 0 "#PWR011" H 2850 5850 50  0001 C CNN
+F 0 "#PWR15" H 2850 5850 50  0001 C CNN
 F 1 "VCC" H 2867 6173 50  0000 C CNN
 F 2 "" H 2850 6000 50  0000 C CNN
@@
 $EndComp
 $Comp
-L GND #PWR012
+L GND #PWR17
 U 1 1 5764558A
 P 2850 6250
-F 0 "#PWR012" H 2850 6000 50  0001 C CNN
+F 0 "#PWR17" H 2850 6000 50  0001 C CNN
 F 1 "GND" H 2855 6077 50  0000 C CNN
 F 2 "" H 2850 6250 50  0000 C CNN
@@
 	1700 5450 1650 5450
 $Comp
-L VAA #PWR013
+L VAA #PWR10
 U 1 1 576834F6
 P 1400 5100
-F 0 "#PWR013" H 1400 4950 50  0001 C CNN
+F 0 "#PWR10" H 1400 4950 50  0001 C CNN
 F 1 "VAA" H 1417 5273 50  0000 C CNN
 F 2 "" H 1400 5100 50  0000 C CNN
@@
 $EndComp
 $Comp
-L VCC #PWR014
+L VCC #PWR9
 U 1 1 5768359B
 P 1200 5100
-F 0 "#PWR014" H 1200 4950 50  0001 C CNN
+F 0 "#PWR9" H 1200 4950 50  0001 C CNN
 F 1 "VCC" H 1217 5273 50  0000 C CNN
 F 2 "" H 1200 5100 50  0000 C CNN
@@
 Connection ~ 1700 5300
 $Comp
-L VDD #PWR015
+L VDD #PWR19
 U 1 1 57683D2A
 P 2650 7100
-F 0 "#PWR015" H 2650 6950 50  0001 C CNN
+F 0 "#PWR19" H 2650 6950 50  0001 C CNN
 F 1 "VDD" H 2667 7273 50  0000 C CNN
 F 2 "" H 2650 7100 50  0000 C CNN
@@
 $EndComp
 $Comp
-L VDD #PWR016
+L VDD #PWR16
 U 1 1 57684056
 P 3750 6000
-F 0 "#PWR016" H 3750 5850 50  0001 C CNN
+F 0 "#PWR16" H 3750 5850 50  0001 C CNN
 F 1 "VDD" H 3767 6173 50  0000 C CNN
 F 2 "" H 3750 6000 50  0000 C CNN
@@
 $EndComp
 $Comp
-L GND #PWR017
+L GND #PWR18
 U 1 1 576840F7
 P 3750 6250
-F 0 "#PWR017" H 3750 6000 50  0001 C CNN
+F 0 "#PWR18" H 3750 6000 50  0001 C CNN
 F 1 "GND" H 3755 6077 50  0000 C CNN
 F 2 "" H 3750 6250 50  0000 C CNN
@@
 	3750 6150 3750 6250
 $Comp
-L VEE #PWR018
+L VEE #PWR2
 U 1 1 57683180
 P 5500 1800
-F 0 "#PWR018" H 5500 1650 50  0001 C CNN
+F 0 "#PWR2" H 5500 1650 50  0001 C CNN
 F 1 "VEE" H 5517 1973 50  0000 C CNN
 F 2 "" H 5500 1800 50  0000 C CNN
@@
 $EndComp
 $Comp
-L GND #PWR019
+L GND #PWR25
 U 1 1 576848A6
 P 4350 7750
-F 0 "#PWR019" H 4350 7500 50  0001 C CNN
+F 0 "#PWR25" H 4350 7500 50  0001 C CNN
 F 1 "GND" H 4355 7577 50  0000 C CNN
 F 2 "" H 4350 7750 50  0000 C CNN
@@
 3V3
 $Comp
-L GND #PWR020
+L GND #PWR6
 U 1 1 577150E0
 P 6350 2450
-F 0 "#PWR020" H 6350 2200 50  0001 C CNN
+F 0 "#PWR6" H 6350 2200 50  0001 C CNN
 F 1 "GND" H 6355 2277 50  0000 C CNN
 F 2 "" H 6350 2450 50  0000 C CNN
@@
 	6350 2400 6800 2400
 $Comp
-L VDD #PWR021
+L VDD #PWR4
 U 1 1 577153D8
 P 6750 2250
-F 0 "#PWR021" H 6750 2100 50  0001 C CNN
+F 0 "#PWR4" H 6750 2100 50  0001 C CNN
 F 1 "VDD" H 6767 2423 50  0000 C CNN
 F 2 "" H 6750 2250 50  0000 C CNN
@@
 	6750 2300 6800 2300
 $Comp
-L VEE #PWR022
+L VEE #PWR5
 U 1 1 57715626
 P 9800 2250
-F 0 "#PWR022" H 9800 2100 50  0001 C CNN
+F 0 "#PWR5" H 9800 2100 50  0001 C CNN
 F 1 "VEE" H 9817 2423 50  0000 C CNN
 F 2 "" H 9800 2250 50  0000 C CNN
@@
 	9800 2400 9800 2250
 $Comp
-L PWR_FLAG #FLG023
+L PWR_FLAG #FLG1
 U 1 1 577166D7
 P 5750 2000
-F 0 "#FLG023" H 5750 2095 50  0001 C CNN
+F 0 "#FLG1" H 5750 2095 50  0001 C CNN
 F 1 "PWR_FLAG" H 5750 2224 50  0000 C CNN
 F 2 "" H 5750 2000 50  0000 C CNN
@@
 Connection ~ 5500 2100
 $Comp
-L PWR_FLAG #FLG024
+L PWR_FLAG #FLG3
 U 1 1 57716880
 P 2100 5200
-F 0 "#FLG024" H 2100 5295 50  0001 C CNN
+F 0 "#FLG3" H 2100 5295 50  0001 C CNN
 F 1 "PWR_FLAG" H 2100 5424 50  0000 C CNN
 F 2 "" H 2100 5200 50  0000 C CNN
@@
 Connection ~ 1850 5300
 $Comp
-L PWR_FLAG #FLG025
+L PWR_FLAG #FLG2
 U 1 1 57716C30
 P 6050 2100
-F 0 "#FLG025" H 6050 2195 50  0001 C CNN
+F 0 "#FLG2" H 6050 2195 50  0001 C CNN
 F 1 "PWR_FLAG" H 6050 2324 50  0000 C CNN
 F 2 "" H 6050 2100 50  0000 C CNN
@@
 	6050 2200 6050 2100
 $Comp
-L PWR_FLAG #FLG026
+L PWR_FLAG #FLG4
 U 1 1 57716DFC
 P 900 5300
-F 0 "#FLG026" H 900 5395 50  0001 C CNN
+F 0 "#FLG4" H 900 5395 50  0001 C CNN
 F 1 "PWR_FLAG" H 900 5524 50  0000 C CNN
 F 2 "" H 900 5300 50  0000 C CNN
@@
 	900  5300 900  5450
 Connection ~ 1200 5450
+$Comp
+L 10uF C3
+U 1 1 5788FFF4
+P 6150 4950
+F 0 "C3" H 6265 4980 40  0000 L CNN
+F 1 "10uF" H 6150 4950 30  0000 C CNN
+F 2 "modular_device_teensy:SM1210" H 6188 4800 30  0001 C CNN
+F 3 "" H 6150 4950 60  0000 C CNN
+F 4 "digikey" H 6250 5150 60  0001 C CNN "Vendor"
+F 5 "445-4536-1-ND" H 6350 5250 60  0001 C CNN "PartNumber"
+F 6 "CAP CER 10UF 50V 10% X7S 1210" H 6450 5350 60  0001 C CNN "Description"
+	1    6150 4950
+	1    0    0    -1
+$EndComp
+$Comp
+L 10uF C4
+U 1 1 5789010A
+P 6600 4950
+F 0 "C4" H 6715 4980 40  0000 L CNN
+F 1 "10uF" H 6600 4950 30  0000 C CNN
+F 2 "modular_device_teensy:SM1210" H 6638 4800 30  0001 C CNN
+F 3 "" H 6600 4950 60  0000 C CNN
+F 4 "digikey" H 6700 5150 60  0001 C CNN "Vendor"
+F 5 "445-4536-1-ND" H 6800 5250 60  0001 C CNN "PartNumber"
+F 6 "CAP CER 10UF 50V 10% X7S 1210" H 6900 5350 60  0001 C CNN "Description"
+	1    6600 4950
+	1    0    0    -1
+$EndComp
+$Comp
+L 10uF C5
+U 1 1 57890173
+P 7050 4950
+F 0 "C5" H 7165 4980 40  0000 L CNN
+F 1 "10uF" H 7050 4950 30  0000 C CNN
+F 2 "modular_device_teensy:SM1210" H 7088 4800 30  0001 C CNN
+F 3 "" H 7050 4950 60  0000 C CNN
+F 4 "digikey" H 7150 5150 60  0001 C CNN "Vendor"
+F 5 "445-4536-1-ND" H 7250 5250 60  0001 C CNN "PartNumber"
+F 6 "CAP CER 10UF 50V 10% X7S 1210" H 7350 5350 60  0001 C CNN "Description"
+	1    7050 4950
+	1    0    0    -1
+$EndComp
+$Comp
+L VDD #PWR7
+U 1 1 578902C2
+P 6150 4700
+F 0 "#PWR7" H 6150 4550 50  0001 C CNN
+F 1 "VDD" H 6167 4873 50  0000 C CNN
+F 2 "" H 6150 4700 50  0000 C CNN
+F 3 "" H 6150 4700 50  0000 C CNN
+	1    6150 4700
+	1    0    0    -1
+$EndComp
+$Comp
+L VEE #PWR8
+U 1 1 57890499
+P 6600 4700
+F 0 "#PWR8" H 6600 4550 50  0001 C CNN
+F 1 "VEE" H 6617 4873 50  0000 C CNN
+F 2 "" H 6600 4700 50  0000 C CNN
+F 3 "" H 6600 4700 50  0000 C CNN
+	1    6600 4700
+	1    0    0    -1
+$EndComp
+Wire Wire Line
+	7050 4750 7050 4700
+Wire Wire Line
+	7050 4700 7100 4700
+Wire Wire Line
+	6150 4700 6150 4750
+Wire Wire Line
+	6600 4700 6600 4750
+Text Label 7100 4700 0    60   ~ 0
+3V3
+$Comp
+L GND #PWR11
+U 1 1 57890974
+P 6150 5200
+F 0 "#PWR11" H 6150 4950 50  0001 C CNN
+F 1 "GND" H 6155 5027 50  0000 C CNN
+F 2 "" H 6150 5200 50  0000 C CNN
+F 3 "" H 6150 5200 50  0000 C CNN
+	1    6150 5200
+	1    0    0    -1
+$EndComp
+$Comp
+L GND #PWR12
+U 1 1 57890A97
+P 6600 5200
+F 0 "#PWR12" H 6600 4950 50  0001 C CNN
+F 1 "GND" H 6605 5027 50  0000 C CNN
+F 2 "" H 6600 5200 50  0000 C CNN
+F 3 "" H 6600 5200 50  0000 C CNN
+	1    6600 5200
+	1    0    0    -1
+$EndComp
+$Comp
+L GND #PWR13
+U 1 1 57890ADE
+P 7050 5200
+F 0 "#PWR13" H 7050 4950 50  0001 C CNN
+F 1 "GND" H 7055 5027 50  0000 C CNN
+F 2 "" H 7050 5200 50  0000 C CNN
+F 3 "" H 7050 5200 50  0000 C CNN
+	1    7050 5200
+	1    0    0    -1
+$EndComp
+Wire Wire Line
+	6150 5150 6150 5200
+Wire Wire Line
+	6600 5150 6600 5200
+Wire Wire Line
+	7050 5150 7050 5200
 $EndSCHEMATC

Commit message: Updated component.
Parts:
- MDT1: footprint modular_device_teensy:MODULAR_DEVICE_TEENSY -> footprints:MODULAR_DEVICE_TEENSY
Changed lines of the file:
@@
 	3850 7100 3850 7250
 $Comp
-L GND #PWR24
+L GND #PWR01
 U 1 1 5751CFDE
 P 3250 7750
-F 0 "#PWR24" H 3250 7500 50  0001 C CNN
+F 0 "#PWR01" H 3250 7500 50  0001 C CNN
 F 1 "GND" H 3255 7577 50  0000 C CNN
 F 2 "" H 3250 7750 50  0000 C CNN
@@
 $EndComp
 $Comp
-L PWR_FLAG #FLG6
+L PWR_FLAG #FLG02
 U 1 1 5751E700
 P 700 7400
-F 0 "#FLG6" H 700 7495 50  0001 C CNN
+F 0 "#FLG02" H 700 7495 50  0001 C CNN
 F 1 "PWR_FLAG" H 700 7624 50  0000 C CNN
 F 2 "" H 700 7400 50  0000 C CNN
@@
 $EndComp
 $Comp
-L PWR_FLAG #FLG5
+L PWR_FLAG #FLG03
 U 1 1 5751E72B
 P 1000 7300
-F 0 "#FLG5" H 1000 7395 50  0001 C CNN
+F 0 "#FLG03" H 1000 7395 50  0001 C CNN
 F 1 "PWR_FLAG" H 1000 7524 50  0000 C CNN
 F 2 "" H 1000 7300 50  0000 C CNN
@@
 $EndComp
 $Comp
-L VAA #PWR21
+L VAA #PWR04
 U 1 1 5751E779
 P 1150 7350
-F 0 "#PWR21" H 1150 7200 50  0001 C CNN
+F 0 "#PWR04" H 1150 7200 50  0001 C CNN
 F 1 "VAA" H 1167 7523 50  0000 C CNN
 F 2 "" H 1150 7350 50  0000 C CNN
@@
 	700  7500 1250 7500
 $Comp
-L GND #PWR22
+L GND #PWR05
 U 1 1 5751E825
 P 1150 7550
-F 0 "#PWR22" H 1150 7300 50  0001 C CNN
+F 0 "#PWR05" H 1150 7300 50  0001 C CNN
 F 1 "GND" H 1155 7377 50  0000 C CNN
 F 2 "" H 1150 7550 50  0000 C CNN
@@
 Connection ~ 1150 7500
 $Comp
-L GND #PWR3
+L GND #PWR06
 U 1 1 5751EC8F
 P 1500 2200
-F 0 "#PWR3" H 1500 1950 50  0001 C CNN
+F 0 "#PWR06" H 1500 1950 50  0001 C CNN
 F 1 "GND" H 1505 2027 50  0000 C CNN
 F 2 "" H 1500 2200 50  0000 C CNN
@@
 $EndComp
 $Comp
-L GND #PWR23
+L GND #PWR07
 U 1 1 5751FC2B
 P 5850 7550
-F 0 "#PWR23" H 5850 7300 50  0001 C CNN
+F 0 "#PWR07" H 5850 7300 50  0001 C CNN
 F 1 "GND" H 5855 7377 50  0000 C CNN
 F 2 "" H 5850 7550 50  0000 C CNN
@@
 	4800 2100 5750 2100
 $Comp
-L +5V #PWR20
+L +5V #PWR08
 U 1 1 57520478
 P 3850 7100
-F 0 "#PWR20" H 3850 6950 50  0001 C CNN
+F 0 "#PWR08" H 3850 6950 50  0001 C CNN
 F 1 "+5V" H 3865 7273 50  0000 C CNN
 F 2 "" H 3850 7100 50  0000 C CNN
@@
 Connection ~ 4950 2100
 $Comp
-L +5V #PWR1
+L +5V #PWR09
 U 1 1 57520888
 P 5300 1800
-F 0 "#PWR1" H 5300 1650 50  0001 C CNN
+F 0 "#PWR09" H 5300 1650 50  0001 C CNN
 F 1 "+5V" H 5315 1973 50  0000 C CNN
 F 2 "" H 5300 1800 50  0000 C CNN
@@
 $EndComp
 $Comp
-L VDD #PWR14
+L VDD #PWR010
 U 1 1 576452DC
 P 1850 5250
-F 0 "#PWR14" H 1850 5100 50  0001 C CNN
+F 0 "#PWR010" H 1850 5100 50  0001 C CNN
 F 1 "VDD" H 1867 5423 50  0000 C CNN
 F 2 "" H 1850 5250 50  0000 C CNN
@@
 $EndComp
 $Comp
-L VCC #PWR15
+L VCC #PWR011
 U 1 1 57645344
 P 2850 6000
-F 0 "#PWR15" H 2850 5850 50  0001 C CNN
+F 0 "#PWR011" H 2850 5850 50  0001 C CNN
 F 1 "VCC" H 2867 6173 50  0000 C CNN
 F 2 "" H 2850 6000 50  0000 C CNN
@@
 $EndComp
 $Comp
-L GND #PWR17
+L GND #PWR012
 U 1 1 5764558A
 P 2850 6250
-F 0 "#PWR17" H 2850 6000 50  0001 C CNN
+F 0 "#PWR012" H 2850 6000 50  0001 C CNN
 F 1 "GND" H 2855 6077 50  0000 C CNN
 F 2 "" H 2850 6250 50  0000 C CNN
@@
 	1700 5450 1650 5450
 $Comp
-L VAA #PWR10
+L VAA #PWR013
 U 1 1 576834F6
 P 1400 5100
-F 0 "#PWR10" H 1400 4950 50  0001 C CNN
+F 0 "#PWR013" H 1400 4950 50  0001 C CNN
 F 1 "VAA" H 1417 5273 50  0000 C CNN
 F 2 "" H 1400 5100 50  0000 C CNN
@@
 $EndComp
 $Comp
-L VCC #PWR9
+L VCC #PWR014
 U 1 1 5768359B
 P 1200 5100
-F 0 "#PWR9" H 1200 4950 50  0001 C CNN
+F 0 "#PWR014" H 1200 4950 50  0001 C CNN
 F 1 "VCC" H 1217 5273 50  0000 C CNN
 F 2 "" H 1200 5100 50  0000 C CNN
@@
 Connection ~ 1700 5300
 $Comp
-L VDD #PWR19
+L VDD #PWR015
 U 1 1 57683D2A
 P 2650 7100
-F 0 "#PWR19" H 2650 6950 50  0001 C CNN
+F 0 "#PWR015" H 2650 6950 50  0001 C CNN
 F 1 "VDD" H 2667 7273 50  0000 C CNN
 F 2 "" H 2650 7100 50  0000 C CNN
@@
 $EndComp
 $Comp
-L VDD #PWR16
+L VDD #PWR016
 U 1 1 57684056
 P 3750 6000
-F 0 "#PWR16" H 3750 5850 50  0001 C CNN
+F 0 "#PWR016" H 3750 5850 50  0001 C CNN
 F 1 "VDD" H 3767 6173 50  0000 C CNN
 F 2 "" H 3750 6000 50  0000 C CNN
@@
 $EndComp
 $Comp
-L GND #PWR18
+L GND #PWR017
 U 1 1 576840F7
 P 3750 6250
-F 0 "#PWR18" H 3750 6000 50  0001 C CNN
+F 0 "#PWR017" H 3750 6000 50  0001 C CNN
 F 1 "GND" H 3755 6077 50  0000 C CNN
 F 2 "" H 3750 6250 50  0000 C CNN
@@
 	3750 6150 3750 6250
 $Comp
-L VEE #PWR2
+L VEE #PWR018
 U 1 1 57683180
 P 5500 1800
-F 0 "#PWR2" H 5500 1650 50  0001 C CNN
+F 0 "#PWR018" H 5500 1650 50  0001 C CNN
 F 1 "VEE" H 5517 1973 50  0000 C CNN
 F 2 "" H 5500 1800 50  0000 C CNN
@@
 $EndComp
 $Comp
-L GND #PWR25
+L GND #PWR019
 U 1 1 576848A6
 P 4350 7750
-F 0 "#PWR25" H 4350 7500 50  0001 C CNN
+F 0 "#PWR019" H 4350 7500 50  0001 C CNN
 F 1 "GND" H 4355 7577 50  0000 C CNN
 F 2 "" H 4350 7750 50  0000 C CNN
@@
 Text Label 9500 3800 0    60   ~ 0
 DAC
-$Comp
-L MODULAR_DEVICE_TEENSY MDT1
-U 1 1 57714506
-P 8050 3050
-F 0 "MDT1" H 8050 4047 60  0000 C CNN
-F 1 "MODULAR_DEVICE_TEENSY" H 8050 3941 60  0000 C CNN
-F 2 "modular_device_teensy:MODULAR_DEVICE_TEENSY" H 8050 4100 60  0001 C CNN
-F 3 "" H 8100 5800 60  0000 C CNN
-F 4 "digikey" H 8050 4200 60  0001 C CNN "Vendor"
-F 5 "S7049-ND" H 8050 4300 60  0001 C CNN "PartNumber"
-F 6 "16 Position Header Through Hole" H 8050 4400 60  0001 C CNN "Description"
-	1    8050 3050
-	1    0    0    -1
-$EndComp
 Wire Wire Line
 	2300 2000 1950 2000
@@
 3V3
 $Comp
-L GND #PWR6
+L GND #PWR020
 U 1 1 577150E0
 P 6350 2450
-F 0 "#PWR6" H 6350 2200 50  0001 C CNN
+F 0 "#PWR020" H 6350 2200 50  0001 C CNN
 F 1 "GND" H 6355 2277 50  0000 C CNN
 F 2 "" H 6350 2450 50  0000 C CNN
@@
 	6350 2400 6800 2400
 $Comp
-L VDD #PWR4
+L VDD #PWR021
 U 1 1 577153D8
 P 6750 2250
-F 0 "#PWR4" H 6750 2100 50  0001 C CNN
+F 0 "#PWR021" H 6750 2100 50  0001 C CNN
 F 1 "VDD" H 6767 2423 50  0000 C CNN
 F 2 "" H 6750 2250 50  0000 C CNN
@@
 	6750 2300 6800 2300
 $Comp
-L VEE #PWR5
+L VEE #PWR022
 U 1 1 57715626
 P 9800 2250
-F 0 "#PWR5" H 9800 2100 50  0001 C CNN
+F 0 "#PWR022" H 9800 2100 50  0001 C CNN
 F 1 "VEE" H 9817 2423 50  0000 C CNN
 F 2 "" H 9800 2250 50  0000 C CNN
@@
 	9800 2400 9800 2250
 $Comp
-L PWR_FLAG #FLG1
+L PWR_FLAG #FLG023
 U 1 1 577166D7
 P 5750 2000
-F 0 "#FLG1" H 5750 2095 50  0001 C CNN
+F 0 "#FLG023" H 5750 2095 50  0001 C CNN
 F 1 "PWR_FLAG" H 5750 2224 50  0000 C CNN
 F 2 "" H 5750 2000 50  0000 C CNN
@@
 Connection ~ 5500 2100
 $Comp
-L PWR_FLAG #FLG3
+L PWR_FLAG #FLG024
 U 1 1 57716880
 P 2100 5200
-F 0 "#FLG3" H 2100 5295 50  0001 C CNN
+F 0 "#FLG024" H 2100 5295 50  0001 C CNN
 F 1 "PWR_FLAG" H 2100 5424 50  0000 C CNN
 F 2 "" H 2100 5200 50  0000 C CNN
@@
 Connection ~ 1850 5300
 $Comp
-L PWR_FLAG #FLG2
+L PWR_FLAG #FLG025
 U 1 1 57716C30
 P 6050 2100
-F 0 "#FLG2" H 6050 2195 50  0001 C CNN
+F 0 "#FLG025" H 6050 2195 50  0001 C CNN
 F 1 "PWR_FLAG" H 6050 2324 50  0000 C CNN
 F 2 "" H 6050 2100 50  0000 C CNN
@@
 	6050 2200 6050 2100
 $Comp
-L PWR_FLAG #FLG4
+L PWR_FLAG #FLG026
 U 1 1 57716DFC
 P 900 5300
-F 0 "#FLG4" H 900 5395 50  0001 C CNN
+F 0 "#FLG026" H 900 5395 50  0001 C CNN
 F 1 "PWR_FLAG" H 900 5524 50  0000 C CNN
 F 2 "" H 900 5300 50  0000 C CNN
@@
 $EndComp
 $Comp
-L VDD #PWR7
+L VDD #PWR027
 U 1 1 578902C2
 P 6150 4700
-F 0 "#PWR7" H 6150 4550 50  0001 C CNN
+F 0 "#PWR027" H 6150 4550 50  0001 C CNN
 F 1 "VDD" H 6167 4873 50  0000 C CNN
 F 2 "" H 6150 4700 50  0000 C CNN
@@
 $EndComp
 $Comp
-L VEE #PWR8
+L VEE #PWR028
 U 1 1 57890499
 P 6600 4700
-F 0 "#PWR8" H 6600 4550 50  0001 C CNN
+F 0 "#PWR028" H 6600 4550 50  0001 C CNN
 F 1 "VEE" H 6617 4873 50  0000 C CNN
 F 2 "" H 6600 4700 50  0000 C CNN
@@
 3V3
 $Comp
-L GND #PWR11
+L GND #PWR029
 U 1 1 57890974
 P 6150 5200
-F 0 "#PWR11" H 6150 4950 50  0001 C CNN
+F 0 "#PWR029" H 6150 4950 50  0001 C CNN
 F 1 "GND" H 6155 5027 50  0000 C CNN
 F 2 "" H 6150 5200 50  0000 C CNN
@@
 $EndComp
 $Comp
-L GND #PWR12
+L GND #PWR030
 U 1 1 57890A97
 P 6600 5200
-F 0 "#PWR12" H 6600 4950 50  0001 C CNN
+F 0 "#PWR030" H 6600 4950 50  0001 C CNN
 F 1 "GND" H 6605 5027 50  0000 C CNN
 F 2 "" H 6600 5200 50  0000 C CNN
@@
 $EndComp
 $Comp
-L GND #PWR13
+L GND #PWR031
 U 1 1 57890ADE
 P 7050 5200
-F 0 "#PWR13" H 7050 4950 50  0001 C CNN
+F 0 "#PWR031" H 7050 4950 50  0001 C CNN
 F 1 "GND" H 7055 5027 50  0000 C CNN
 F 2 "" H 7050 5200 50  0000 C CNN
@@
 Wire Wire Line
 	7050 5150 7050 5200
+$Comp
+L MODULAR_DEVICE_TEENSY MDT1
+U 1 1 578CF1A5
+P 8050 3050
+F 0 "MDT1" H 8050 4047 60  0000 C CNN
+F 1 "MODULAR_DEVICE_TEENSY" H 8050 3941 60  0000 C CNN
+F 2 "footprints:MODULAR_DEVICE_TEENSY" H 8050 4100 60  0001 C CNN
+F 3 "" H 8100 5800 60  0000 C CNN
+F 4 "digikey" H 8050 4200 60  0001 C CNN "Vendor"
+F 5 "S7049-ND" H 8050 4300 60  0001 C CNN "PartNumber"
+F 6 "16 Position Header Through Hole" H 8050 4400 60  0001 C CNN "Description"
+	1    8050 3050
+	1    0    0    -1
+$EndComp
 $EndSCHEMATC

Commit message: Finished pcb v1.0.
Parts:
- MDT1: footprint footprints:MODULAR_DEVICE_TEENSY -> modular_device_teensy:MODULAR_DEVICE_TEENSY; PartCount (none) -> 2
Changed lines of the file:
@@
 LIBS:components
 LIBS:modular_device_teensy
-LIBS:modular_device_teensy-cache
 EELAYER 25 0
 EELAYER END
@@
 $Comp
 L MODULAR_DEVICE_TEENSY MDT1
-U 1 1 578CF1A5
+U 1 1 578D0E11
 P 8050 3050
 F 0 "MDT1" H 8050 4047 60  0000 C CNN
 F 1 "MODULAR_DEVICE_TEENSY" H 8050 3941 60  0000 C CNN
-F 2 "footprints:MODULAR_DEVICE_TEENSY" H 8050 4100 60  0001 C CNN
+F 2 "modular_device_teensy:MODULAR_DEVICE_TEENSY" H 8050 4100 60  0001 C CNN
 F 3 "" H 8100 5800 60  0000 C CNN
 F 4 "digikey" H 8050 4200 60  0001 C CNN "Vendor"
 F 5 "S7049-ND" H 8050 4300 60  0001 C CNN "PartNumber"
 F 6 "16 Position Header Through Hole" H 8050 4400 60  0001 C CNN "Description"
+F 7 "2" H 9350 4300 60  0001 C CNN "PartCount"
 	1    8050 3050
 	1    0    0    -1
