File: pcb/modular_device_teensy.sch (KiCad schematic (older format))
At the start: 20 parts, among them P1 PWR_JACK_2.5x5.5_SMD_RA, P2 HEADER_01X03_SMD_RA, P3 HEADER_01X03_SMD_RA, P4 HEADER_01X03_SMD_RA, P5 BNC_DOUBLE_RA, P6 HEADER_01X02_SMD_RA, P7 HEADER_01X02_SMD_RA, SW1 KT_SWITCH

Commit message: Progress towards v1.1.
Parts:
- removed MDT1: MODULAR_DEVICE_TEENSY, modular_device_teensy:MODULAR_DEVICE_TEENSY, symbol MODULAR_DEVICE_TEENSY
- added MDT1: MODULAR_DEVICE_TEENSY_FEMALE, modular_device_teensy:MODULAR_DEVICE_TEENSY, symbol MODULAR_DEVICE_TEENSY_FEMALE
Changed lines of the file:
@@
 LIBS:components
 LIBS:modular_device_teensy
+LIBS:modular_device_teensy-cache
 EELAYER 25 0
 EELAYER END
@@
 Title "modular_device_teensy"
 Date ""
-Rev "1.0"
+Rev "1.1"
 Comp "Janelia"
 Comment1 ""
@@
 	7050 5150 7050 5200
 $Comp
-L MODULAR_DEVICE_TEENSY MDT1
-U 1 1 578D0E11
+L MODULAR_DEVICE_TEENSY_FEMALE MDT1
+U 1 1 578F97D8
 P 8050 3050
 F 0 "MDT1" H 8050 4047 60  0000 C CNN
-F 1 "MODULAR_DEVICE_TEENSY" H 8050 3941 60  0000 C CNN
+F 1 "MODULAR_DEVICE_TEENSY_FEMALE" H 8050 3941 60  0000 C CNN
 F 2 "modular_device_teensy:MODULAR_DEVICE_TEENSY" H 8050 4100 60  0001 C CNN
 F 3 "" H 8100 5800 60  0000 C CNN
 F 4 "digikey" H 8050 4200 60  0001 C CNN "Vendor"
 F 5 "S7049-ND" H 8050 4300 60  0001 C CNN "PartNumber"
-F 6 "16 Position Header Through Hole" H 8050 4400 60  0001 C CNN "Description"
+F 6 "16 Position Header Through Hole Female Socket" H 8050 4400 60  0001 C CNN "Description"
 F 7 "2" H 9350 4300 60  0001 C CNN "PartCount"
 	1    8050 3050

Commit message: More progress towards pcb v1.1.
Parts:
- added MH1, MH2, MH3: MNT_HOLE, modular_device_teensy:MOUNTING_HOLE_4-40, symbol MNT_HOLE
Connections:
- no-connect marks 5 -> 8
Changed lines of the file:
@@
 	1    0    0    -1
 $EndComp
+$Comp
+L MNT_HOLE MH1
+U 1 1 57928CA5
+P 8900 4700
+F 0 "MH1" H 8977 4741 50  0000 L CNN
+F 1 "MNT_HOLE" H 8977 4650 50  0000 L CNN
+F 2 "modular_device_teensy:MOUNTING_HOLE_4-40" H 8800 4700 50  0001 C CNN
+F 3 "" H 8900 4700 50  0000 C CNN
+F 4 "digikey" H 9000 4900 60  0001 C CNN "Vendor"
+F 5 "36-3480-ND" H 9100 5000 60  0001 C CNN "PartNumber"
+F 6 "Round Standoff Threaded 4-40 Aluminum 0.500in" H 9200 5100 60  0001 C CNN "Description"
+	1    8900 4700
+	1    0    0    -1
+$EndComp
+$Comp
+L MNT_HOLE MH2
+U 1 1 57928DFF
+P 8900 4900
+F 0 "MH2" H 8977 4941 50  0000 L CNN
+F 1 "MNT_HOLE" H 8977 4850 50  0000 L CNN
+F 2 "modular_device_teensy:MOUNTING_HOLE_4-40" H 8800 4900 50  0001 C CNN
+F 3 "" H 8900 4900 50  0000 C CNN
+F 4 "digikey" H 9000 5100 60  0001 C CNN "Vendor"
+F 5 "36-3480-ND" H 9100 5200 60  0001 C CNN "PartNumber"
+F 6 "Round Standoff Threaded 4-40 Aluminum 0.500in" H 9200 5300 60  0001 C CNN "Description"
+	1    8900 4900
+	1    0    0    -1
+$EndComp
+$Comp
+L MNT_HOLE MH3
+U 1 1 57928E5B
+P 8900 5100
+F 0 "MH3" H 8977 5141 50  0000 L CNN
+F 1 "MNT_HOLE" H 8977 5050 50  0000 L CNN
+F 2 "modular_device_teensy:MOUNTING_HOLE_4-40" H 8800 5100 50  0001 C CNN
+F 3 "" H 8900 5100 50  0000 C CNN
+F 4 "digikey" H 9000 5300 60  0001 C CNN "Vendor"
+F 5 "36-3480-ND" H 9100 5400 60  0001 C CNN "PartNumber"
+F 6 "Round Standoff Threaded 4-40 Aluminum 0.500in" H 9200 5500 60  0001 C CNN "Description"
+	1    8900 5100
+	1    0    0    -1
+$EndComp
+NoConn ~ 8700 4700
+NoConn ~ 8700 4900
+NoConn ~ 8700 5100
 $EndSCHEMATC

Commit message: Modified mounting hole spacer diameter.
Parts:
- MH1, MH2, MH3: Description Round Standoff Threaded 4-40 Aluminum 0.500in -> Round Standoff Threaded 4-40 Aluminum 0.500in 0.187in; PartNumber 36-3480-ND -> 36-2027-ND
Changed lines of the file:
@@
 	1    0    0    -1
 $EndComp
+NoConn ~ 8700 4700
+NoConn ~ 8700 4900
+NoConn ~ 8700 5100
 $Comp
 L MNT_HOLE MH1
-U 1 1 57928CA5
+U 1 1 57967F84
 P 8900 4700
 F 0 "MH1" H 8977 4741 50  0000 L CNN
@@
 F 3 "" H 8900 4700 50  0000 C CNN
 F 4 "digikey" H 9000 4900 60  0001 C CNN "Vendor"
-F 5 "36-3480-ND" H 9100 5000 60  0001 C CNN "PartNumber"
-F 6 "Round Standoff Threaded 4-40 Aluminum 0.500in" H 9200 5100 60  0001 C CNN "Description"
+F 5 "36-2027-ND" H 9100 5000 60  0001 C CNN "PartNumber"
+F 6 "Round Standoff Threaded 4-40 Aluminum 0.500in 0.187in" H 9200 5100 60  0001 C CNN "Description"
 	1    8900 4700
 	1    0    0    -1
@@
 $Comp
 L MNT_HOLE MH2
-U 1 1 57928DFF
+U 1 1 57968003
 P 8900 4900
 F 0 "MH2" H 8977 4941 50  0000 L CNN
@@
 F 3 "" H 8900 4900 50  0000 C CNN
 F 4 "digikey" H 9000 5100 60  0001 C CNN "Vendor"
-F 5 "36-3480-ND" H 9100 5200 60  0001 C CNN "PartNumber"
-F 6 "Round Standoff Threaded 4-40 Aluminum 0.500in" H 9200 5300 60  0001 C CNN "Description"
+F 5 "36-2027-ND" H 9100 5200 60  0001 C CNN "PartNumber"
+F 6 "Round Standoff Threaded 4-40 Aluminum 0.500in 0.187in" H 9200 5300 60  0001 C CNN "Description"
 	1    8900 4900
 	1    0    0    -1
@@
 $Comp
 L MNT_HOLE MH3
-U 1 1 57928E5B
+U 1 1 5796805F
 P 8900 5100
 F 0 "MH3" H 8977 5141 50  0000 L CNN
@@
 F 3 "" H 8900 5100 50  0000 C CNN
 F 4 "digikey" H 9000 5300 60  0001 C CNN "Vendor"
-F 5 "36-3480-ND" H 9100 5400 60  0001 C CNN "PartNumber"
-F 6 "Round Standoff Threaded 4-40 Aluminum 0.500in" H 9200 5500 60  0001 C CNN "Description"
+F 5 "36-2027-ND" H 9100 5400 60  0001 C CNN "PartNumber"
+F 6 "Round Standoff Threaded 4-40 Aluminum 0.500in 0.187in" H 9200 5500 60  0001 C CNN "Description"
 	1    8900 5100
 	1    0    0    -1
 $EndComp
-NoConn ~ 8700 4700
-NoConn ~ 8700 4900
-NoConn ~ 8700 5100
 $EndSCHEMATC

Commit message: Switch to new MODULAR_DEVICE_TEENSY footprint.
Parts:
- MDT1: footprint modular_device_teensy:MODULAR_DEVICE_TEENSY -> footprints:MODULAR_DEVICE_TEENSY_FEMALE
Changed lines of the file:
@@
 Wire Wire Line
 	7050 5150 7050 5200
-$Comp
-L MODULAR_DEVICE_TEENSY_FEMALE MDT1
-U 1 1 578F97D8
-P 8050 3050
-F 0 "MDT1" H 8050 4047 60  0000 C CNN
-F 1 "MODULAR_DEVICE_TEENSY_FEMALE" H 8050 3941 60  0000 C CNN
-F 2 "modular_device_teensy:MODULAR_DEVICE_TEENSY" H 8050 4100 60  0001 C CNN
-F 3 "" H 8100 5800 60  0000 C CNN
-F 4 "digikey" H 8050 4200 60  0001 C CNN "Vendor"
-F 5 "S7049-ND" H 8050 4300 60  0001 C CNN "PartNumber"
-F 6 "16 Position Header Through Hole Female Socket" H 8050 4400 60  0001 C CNN "Description"
-F 7 "2" H 9350 4300 60  0001 C CNN "PartCount"
-	1    8050 3050
-	1    0    0    -1
-$EndComp
 NoConn ~ 8700 4700
 NoConn ~ 8700 4900
@@
 	1    0    0    -1
 $EndComp
+$Comp
+L MODULAR_DEVICE_TEENSY_FEMALE MDT1
+U 1 1 57993352
+P 8050 3050
+F 0 "MDT1" H 8050 4047 60  0000 C CNN
+F 1 "MODULAR_DEVICE_TEENSY_FEMALE" H 8050 3941 60  0000 C CNN
+F 2 "footprints:MODULAR_DEVICE_TEENSY_FEMALE" H 8050 4100 60  0001 C CNN
+F 3 "" H 8100 5800 60  0000 C CNN
+F 4 "digikey" H 8050 4200 60  0001 C CNN "Vendor"
+F 5 "S7049-ND" H 8050 4300 60  0001 C CNN "PartNumber"
+F 6 "16 Position Header Through Hole Female Socket" H 8050 4400 60  0001 C CNN "Description"
+F 7 "2" H 9350 4300 60  0001 C CNN "PartCount"
+	1    8050 3050
+	1    0    0    -1
+$EndComp

Commit message: Finished pcb v1.1.
Parts:
- MDT1: footprint footprints:MODULAR_DEVICE_TEENSY_FEMALE -> modular_device_teensy:MODULAR_DEVICE_TEENSY_FEMALE
Changed lines of the file:
@@
 F 0 "MDT1" H 8050 4047 60  0000 C CNN
 F 1 "MODULAR_DEVICE_TEENSY_FEMALE" H 8050 3941 60  0000 C CNN
-F 2 "footprints:MODULAR_DEVICE_TEENSY_FEMALE" H 8050 4100 60  0001 C CNN
+F 2 "modular_device_teensy:MODULAR_DEVICE_TEENSY_FEMALE" H 8050 4100 60  0001 C CNN
 F 3 "" H 8100 5800 60  0000 C CNN
 F 4 "digikey" H 8050 4200 60  0001 C CNN "Vendor"
